Commit message: Add water to inspection map, make a custom racetrack

File: cpr_inspection_gazebo/urdf/inspection_geometry.urdf.xacro (robot description, xacro)
@@ -11,10 +11,4 @@
       <geometry>
         <mesh filename="package://cpr_inspection_gazebo/meshes/inspection_world.dae" scale="2 2 1"/>
-      </geometry>
-    </visual>
-    <visual>
-      <origin xyz="0 0 0" rpy="0 0 3.141592653589793"/>
-      <geometry>
-        <mesh filename="package://cpr_inspection_gazebo/meshes/inspection_water.dae" scale="2 2 1"/>
       </geometry>
     </visual>
@@ -34,4 +28,66 @@
     </collision>
   </link>
+  <link name="inspection_water_link">
+    <visual>
+      <origin xyz="0 0 0" rpy="0 0 3.141592653589793"/>
+      <geometry>
+        <mesh filename="package://cpr_inspection_gazebo/meshes/inspection_water.dae" scale="2 2 1"/>
+      </geometry>
+    </visual>
+    <visual>
+      <origin xyz="0 0 -0.2" rpy="0 0 3.141592653589793"/>
+      <geometry>
+        <mesh filename="package://cpr_inspection_gazebo/meshes/inspection_water.dae" scale="2 2 1"/>
+      </geometry>
+    </visual>
+    <visual>
+      <origin xyz="0 0 -0.4" rpy="0 0 3.141592653589793"/>
+      <geometry>
+        <mesh filename="package://cpr_inspection_gazebo/meshes/inspection_water.dae" scale="2 2 1"/>
+      </geometry>
+    </visual>
+    <visual>
+      <origin xyz="0 0 -0.6" rpy="0 0 3.141592653589793"/>
+      <geometry>
+        <mesh filename="package://cpr_inspection_gazebo/meshes/inspection_water.dae" scale="2 2 1"/>
+      </geometry>
+    </visual>
+    <visual>
+      <origin xyz="0 0 -0.8" rpy="0 0 3.141592653589793"/>
+      <geometry>
+        <mesh filename="package://cpr_inspection_gazebo/meshes/inspection_water.dae" scale="2 2 1"/>
+      </geometry>
+    </visual>
+    <visual>
+      <origin xyz="0 0 -1.0" rpy="0 0 3.141592653589793"/>
+      <geometry>
+        <mesh filename="package://cpr_inspection_gazebo/meshes/inspection_water.dae" scale="2 2 1"/>
+      </geometry>
+    </visual>
+    <visual>
+      <origin xyz="0 0 -1.2" rpy="0 0 3.141592653589793"/>
+      <geometry>
+        <mesh filename="package://cpr_inspection_gazebo/meshes/inspection_water.dae" scale="2 2 1"/>
+      </geometry>
+    </visual>
+    <visual>
+      <origin xyz="0 0 -1.4" rpy="0 0 3.141592653589793"/>
+      <geometry>
+        <mesh filename="package://cpr_inspection_gazebo/meshes/inspection_water.dae" scale="2 2 1"/>
+      </geometry>
+    </visual>
+    <visual>
+      <origin xyz="0 0 -1.6" rpy="0 0 3.141592653589793"/>
+      <geometry>
+        <mesh filename="package://cpr_inspection_gazebo/meshes/inspection_water.dae" scale="2 2 1"/>
+      </geometry>
+    </visual>
+  </link>
+  <joint name="base_to_water_joint" type="fixed">
+    <parent link="inspection_world_link" />
+    <child link="inspection_water_link" />
+    <origin xyz="0 0 0" rpy="0 0 0" />
+    <axis xyz="0 0 0" />
+  </joint>
   <xacro:include filename="$(find cpr_accessories_gazebo)/urdf/base_station.urdf.xacro" />
   <xacro:cpr_base_station name="base_station" parent="inspection_world_link">

Commit message: Changes to inspection map

File: cpr_inspection_gazebo/urdf/inspection_geometry.urdf.xacro (robot description, xacro)
@@ -29,4 +29,58 @@
   </link>
   <link name="inspection_water_link">
+    <visual>
+      <origin xyz="0 0 0" rpy="3.141592 0 0"/>
+      <geometry>
+        <mesh filename="package://cpr_inspection_gazebo/meshes/inspection_water.dae" scale="2 2 1"/>
+      </geometry>
+    </visual>
+    <visual>
+      <origin xyz="0 0 -0.2" rpy="3.141592 0 0"/>
+      <geometry>
+        <mesh filename="package://cpr_inspection_gazebo/meshes/inspection_water.dae" scale="2 2 1"/>
+      </geometry>
+    </visual>
+    <visual>
+      <origin xyz="0 0 -0.4" rpy="3.141592 0 0"/>
+      <geometry>
+        <mesh filename="package://cpr_inspection_gazebo/meshes/inspection_water.dae" scale="2 2 1"/>
+      </geometry>
+    </visual>
+    <visual>
+      <origin xyz="0 0 -0.6" rpy="3.141592 0 0"/>
+      <geometry>
+        <mesh filename="package://cpr_inspection_gazebo/meshes/inspection_water.dae" scale="2 2 1"/>
+      </geometry>
+    </visual>
+    <visual>
+      <origin xyz="0 0 -0.8" rpy="3.141592 0 0"/>
+      <geometry>
+        <mesh filename="package://cpr_inspection_gazebo/meshes/inspection_water.dae" scale="2 2 1"/>
+      </geometry>
+    </visual>
+    <visual>
+      <origin xyz="0 0 -1.0" rpy="3.141592 0 0"/>
+      <geometry>
+        <mesh filename="package://cpr_inspection_gazebo/meshes/inspection_water.dae" scale="2 2 1"/>
+      </geometry>
+    </visual>
+    <visual>
+      <origin xyz="0 0 -1.2" rpy="3.141592 0 0"/>
+      <geometry>
+        <mesh filename="package://cpr_inspection_gazebo/meshes/inspection_water.dae" scale="2 2 1"/>
+      </geometry>
+    </visual>
+    <visual>
+      <origin xyz="0 0 -1.4" rpy="3.141592 0 0"/>
+      <geometry>
+        <mesh filename="package://cpr_inspection_gazebo/meshes/inspection_water.dae" scale="2 2 1"/>
+      </geometry>
+    </visual>
+    <visual>
+      <origin xyz="0 0 -1.6" rpy="3.141592 0 0"/>
+      <geometry>
+        <mesh filename="package://cpr_inspection_gazebo/meshes/inspection_water.dae" scale="2 2 1"/>
+      </geometry>
+    </visual>
     <visual>
       <origin xyz="0 0 0" rpy="0 0 3.141592653589793"/>
